File: pcb/67_E.kicad_pcb (KiCad board)
At the start: 2 copper layers, 303.2 x 97.6 mm, 123 parts, among them U1 ATmega32U4-AU, U2 SRV05-4, X1 Crystal_GND24_Small

Commit message: Re-trace USB port, fuse and ESD
Parts:
- moved F1 9.43 mm to (82.6, 102.5)
- moved U2 4.12 mm to (76.5, 95.6)
- moved R2 2.35 mm to (78.0, 84.5)
- moved R1 2.31 mm to (75.0, 84.6)
- moved R3 2.31 mm to (85.1, 107.1)
- moved R4 2.31 mm to (83.0, 107.1)
Routing:
- net col13: track 300.5 -> 170.6 mm
- net col1: track 86.9 -> 181.5 mm, vias 2 -> 7
- net (no net): track 367.5 -> 297.8 mm
- net col14: track 284.6 -> 232.4 mm, vias 1 -> 2
- net col15: track 270.2 -> 232.2 mm, vias 1 -> 2
- net Net-(D1-Pad2): track 33.7 -> 0.00 mm, vias 1 -> 0
- net Net-(D23-Pad2): track 18.9 -> 45.6 mm
- net +5V: track 224.3 -> 214.6 mm
- net VCC: track 25.2 -> 33.3 mm
- net Net-(D24-Pad2): track 49.0 -> 45.6 mm
- net Net-(D9-Pad2): track 47.9 -> 45.2 mm, vias 1 -> 2
- net Net-(R1-Pad2): track 5.67 -> 3.21 mm
- net Net-(R3-Pad2): track 121.2 -> 123.5 mm
- net Net-(R4-Pad2): track 122.3 -> 124.6 mm
- net GND: track 31.5 -> 33.8 mm
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
Commit message: finish rerouting switch matrix
Routing:
- net (no net): track 297.8 -> 0.00 mm
- net col13: track 170.6 -> 333.2 mm, vias 1 -> 6
- net col2: track 55.6 -> 168.4 mm, vias 2 -> 7
- net col6: track 19.3 -> 108.8 mm, vias 0 -> 3
- net col5: track 14.6 -> 97.6 mm, vias 0 -> 4
- net col15: track 232.2 -> 295.9 mm, vias 2 -> 5
- net col11: track 226.2 -> 263.2 mm, vias 1 -> 7
- net Net-(D1-Pad2): track 0.00 -> 35.6 mm, vias 0 -> 2
- net col10: track 176.7 -> 206.1 mm, vias 1 -> 5
- net col12: track 248.6 -> 274.8 mm, vias 1 -> 5
- net col3: track 121.5 -> 147.0 mm, vias 1 -> 5
- net col4: track 94.8 -> 119.2 mm, vias 1 -> 5
- net col9: track 161.8 -> 185.5 mm, vias 1 -> 5
- net Net-(D26-Pad2): track 8.17 -> 31.6 mm
- net col8: track 146.7 -> 169.1 mm, vias 1 -> 5
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
Commit message: Add RGB underglow to PCB
Parts:
- added C10: 0.1u, Capacitor_SMD:C_0805_2012Metric, B.Cu at (300.6, 95.3)
- added C11: 0.1u, Capacitor_SMD:C_0805_2012Metric, B.Cu at (200.6, 95.3)
- added C12: 0.1u, Capacitor_SMD:C_0805_2012Metric, B.Cu at (137.2, 95.3)
- added C13: 0.1u, Capacitor_SMD:C_0805_2012Metric, B.Cu at (250.3, 95.3)
- added C14: 0.1u, Capacitor_SMD:C_0805_2012Metric, B.Cu at (83.2, 148.7)
- added C15: 0.1u, Capacitor_SMD:C_0805_2012Metric, B.Cu at (101.2, 95.3)
- added C16: 0.1u, Capacitor_SMD:C_0805_2012Metric, B.Cu at (127.6, 153.3)
- added C17: C, Capacitor_SMD:C_0805_2012Metric, B.Cu at (250.5, 151.8)
- added C18: C, Capacitor_SMD:C_0805_2012Metric, B.Cu at (300.7, 151.8)
- added C19: C, Capacitor_SMD:C_0805_2012Metric, B.Cu at (350.0, 151.8)
- added C20: C, Capacitor_SMD:C_0805_2012Metric, B.Cu at (200.9, 152.1)
- added C6: 0.1u, Capacitor_SMD:C_0805_2012Metric, B.Cu at (350.0, 95.3)
- added D16: WS2812B, LED_SMD:LED_WS2812B_PLCC4_5.0x5.0mm_P3.2mm, B.Cu at (81.7, 152.6)
- added D37: WS2812B, LED_SMD:LED_WS2812B_PLCC4_5.0x5.0mm_P3.2mm, B.Cu at (132.7, 152.6)
- added D38: WS2812B, LED_SMD:LED_WS2812B_PLCC4_5.0x5.0mm_P3.2mm, B.Cu at (196.0, 152.7)
- added D39: WS2812B, LED_SMD:LED_WS2812B_PLCC4_5.0x5.0mm_P3.2mm, B.Cu at (245.6, 152.5)
- added D40: WS2812B, LED_SMD:LED_WS2812B_PLCC4_5.0x5.0mm_P3.2mm, B.Cu at (296.0, 152.5)
- added D41: WS2812B, LED_SMD:LED_WS2812B_PLCC4_5.0x5.0mm_P3.2mm, B.Cu at (345.3, 152.5)
- added D42: WS2812B, LED_SMD:LED_WS2812B_PLCC4_5.0x5.0mm_P3.2mm, B.Cu at (345.3, 95.9)
- added D43: WS2812B, LED_SMD:LED_WS2812B_PLCC4_5.0x5.0mm_P3.2mm, B.Cu at (296.0, 95.9)
- added D44: WS2812B, LED_SMD:LED_WS2812B_PLCC4_5.0x5.0mm_P3.2mm, B.Cu at (245.6, 95.9)
- added D45: WS2812B, LED_SMD:LED_WS2812B_PLCC4_5.0x5.0mm_P3.2mm, B.Cu at (196.0, 95.9)
- added D46: WS2812B, LED_SMD:LED_WS2812B_PLCC4_5.0x5.0mm_P3.2mm, B.Cu at (132.7, 95.9)
- added D47: WS2812B, LED_SMD:LED_WS2812B_PLCC4_5.0x5.0mm_P3.2mm, B.Cu at (96.7, 95.9)
- MX1: footprint MX_Only:MXOnly-2U-Hotswap-LED -> MX_Only:MXOnly-2U-Hotswap
- MX36: value MX-LED -> MX-NoLED
Connections:
- U1 pad 12: (no net) -> LED_DATA
Routing:
- net +5V: track 216.4 -> 778.0 mm, vias 5 -> 9
- net LED_DATA: track 0.00 -> 95.6 mm, vias 0 -> 2
- net Net-(D37-Pad2): track 0.00 -> 84.8 mm, vias 0 -> 2
- net Net-(D41-Pad2): track 0.00 -> 82.4 mm
- net Net-(D45-Pad2): track 0.00 -> 59.8 mm
- net GND: track 37.7 -> 93.5 mm, vias 4 -> 13
- net Net-(D16-Pad2): track 0.00 -> 47.4 mm
- net Net-(D38-Pad2): track 0.00 -> 47.2 mm, vias 0 -> 2
- net Net-(D43-Pad2): track 0.00 -> 46.8 mm
- net Net-(D39-Pad2): track 0.00 -> 46.8 mm
- net Net-(D44-Pad2): track 0.00 -> 46.0 mm
- net Net-(D42-Pad2): track 0.00 -> 46.0 mm
- net Net-(D40-Pad2): track 0.00 -> 45.8 mm
- net Net-(D46-Pad2): track 0.00 -> 33.1 mm
- net col1: track 180.1 -> 183.0 mm
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Other:
- board text added: "67mk_E Hotswap RGB rev.1 by Jakob based on a design from keyboards.elmo.space"
- board text removed: "67mk_E rev.1 keyboards.elmo.space"
- board text removed: "x"

Commit message: wip
Parts:
- added G***: LOGO, custom_parts:vial_logo, B.Cu at (140.1, 115.7)
- added G***: LOGO, custom_parts:qmk, B.Cu at (112.6, 115.6)
- C10, C11, C12, C13, C14, C15, C16, C6: value 0.1u -> 0.1uF
- C17, C18, C19, C20: value C -> 0.1uF
- RESET1: footprint Button_Switch_SMD:SW_SPST_TL3342 -> TestPoint:TestPoint_2Pads_Pitch2.54mm_Drill0.8mm
- X1: value Crystal_GND24_Small -> 16MHz
- moved RESET1 8.01 mm to (225.7, 169.0)
- moved C14 4.68 mm to (87.0, 151.4), turned to 270 degrees
- moved C11 1.80 mm to (202.4, 95.3)
- moved C12 1.65 mm to (138.9, 95.3)
- moved C15 1.44 mm to (102.7, 95.2)
- moved C10 1.44 mm to (302.0, 95.3)
- moved C13 1.32 mm to (251.6, 95.3)
- moved C18 1.23 mm to (301.9, 151.8)
- moved C19 1.23 mm to (351.2, 151.8)
- moved C20 1.22 mm to (202.1, 152.1)
- moved C6 1.21 mm to (351.2, 95.3)
- moved C17 1.17 mm to (251.6, 151.8)
- moved C16 0.98 mm to (126.6, 153.3)
Routing:
- net Net-(R6-Pad1): track 94.8 -> 76.4 mm
- net GND: track 93.5 -> 108.9 mm, vias 13 -> 26
- net +5V: track 778.0 -> 780.6 mm
- net col10: track 206.1 -> 204.8 mm
Other:
- board text added: "JKB"
